Commit message: feat: update description

File: robotiq_ft_sensor_description/urdf/robotiq_ft300.urdf.xacro (robot description, xacro)
@@ -18,5 +18,5 @@
                 <origin xyz="0 0 0" rpy="0 0 0" />
                 <geometry>
-                    <mesh filename="file://$(find robotiq_ft_sensor_description)/meshes/visual/robotiq_ft300.STL"/>
+                    <mesh filename="package://meshes/visual/robotiq_ft300.STL"/>
                 </geometry>
                 <material name="Robotiq-Black">
@@ -27,5 +27,5 @@
                 <origin xyz="0 0 0" rpy="0 0 0" />
                 <geometry>
-                    <mesh filename="file://$(find robotiq_ft_sensor_description)/meshes/collision/robotiq_ft300.STL"/>
+                    <mesh filename="package://meshes/collision/robotiq_ft300.STL"/>
                 </geometry>
             </collision>
@@ -36,5 +36,5 @@
                 <origin xyz="0 0 0" rpy="0 0 0" />
                 <geometry>
-                    <mesh filename="file://$(find robotiq_ft_sensor_description)/meshes/visual/mountings/robotiq_ft300-G-062-COUPLING_G-50-4M6-1D6_20181119.STL"/>
+                    <mesh filename="package://meshes/visual/mountings/robotiq_ft300-G-062-COUPLING_G-50-4M6-1D6_20181119.STL"/>
                 </geometry>
                 <material name="Robotiq-Grey">
@@ -45,5 +45,5 @@
                 <origin xyz="0 0 0" rpy="0 0 0" />
                 <geometry>
-                    <mesh filename="file://$(find robotiq_ft_sensor_description)/meshes/collision/mountings/robotiq_ft300-G-062-COUPLING_G-50-4M6-1D6_20181119.STL"/>
+                    <mesh filename="package://meshes/collision/mountings/robotiq_ft300-G-062-COUPLING_G-50-4M6-1D6_20181119.STL"/>
                 </geometry>
             </collision>

File: robotiq_ft_sensor_description/urdf/robotiq_fts150.urdf.xacro (robot description, xacro)
@@ -18,5 +18,5 @@
                 <origin xyz="0 0 0" rpy="0 0 0" />
                 <geometry>
-                    <mesh filename="file://$(find robotiq_ft_sensor_description)/meshes/visual/robotiq_fts150.stl"/>
+                    <mesh filename="package://meshes/visual/robotiq_fts150.stl"/>
                 </geometry>
                 <material name="black"/>
@@ -25,5 +25,5 @@
                 <origin xyz="0 0 0" rpy="0 0 0" />
                 <geometry>
-                    <mesh filename="file://$(find robotiq_ft_sensor_description)/meshes/collision/robotiq_fts150.stl"/>
+                    <mesh filename="package://meshes/collision/robotiq_fts150.stl"/>
                 </geometry>
             </collision>

Commit message: feat: update description

File: robotiq_ft_sensor_description/urdf/robotiq_ft300.urdf.xacro (robot description, xacro)
@@ -18,5 +18,5 @@
                 <origin xyz="0 0 0" rpy="0 0 0" />
                 <geometry>
-                    <mesh filename="package://meshes/visual/robotiq_ft300.STL"/>
+                    <mesh filename="package://robotiq_ft_sensor_description/meshes/visual/robotiq_ft300.STL"/>
                 </geometry>
                 <material name="Robotiq-Black">
@@ -27,5 +27,5 @@
                 <origin xyz="0 0 0" rpy="0 0 0" />
                 <geometry>
-                    <mesh filename="package://meshes/collision/robotiq_ft300.STL"/>
+                    <mesh filename="package://robotiq_ft_sensor_description/meshes/collision/robotiq_ft300.STL"/>
                 </geometry>
             </collision>
@@ -36,5 +36,5 @@
                 <origin xyz="0 0 0" rpy="0 0 0" />
                 <geometry>
-                    <mesh filename="package://meshes/visual/mountings/robotiq_ft300-G-062-COUPLING_G-50-4M6-1D6_20181119.STL"/>
+                    <mesh filename="package://robotiq_ft_sensor_description/meshes/visual/mountings/robotiq_ft300-G-062-COUPLING_G-50-4M6-1D6_20181119.STL"/>
                 </geometry>
                 <material name="Robotiq-Grey">
@@ -45,5 +45,5 @@
                 <origin xyz="0 0 0" rpy="0 0 0" />
                 <geometry>
-                    <mesh filename="package://meshes/collision/mountings/robotiq_ft300-G-062-COUPLING_G-50-4M6-1D6_20181119.STL"/>
+                    <mesh filename="package://robotiq_ft_sensor_description/meshes/collision/mountings/robotiq_ft300-G-062-COUPLING_G-50-4M6-1D6_20181119.STL"/>
                 </geometry>
             </collision>

File: robotiq_ft_sensor_description/urdf/robotiq_fts150.urdf.xacro (robot description, xacro)
@@ -18,5 +18,5 @@
                 <origin xyz="0 0 0" rpy="0 0 0" />
                 <geometry>
-                    <mesh filename="package://meshes/visual/robotiq_fts150.stl"/>
+                    <mesh filename="package://robotiq_ft_sensor_description/meshes/visual/robotiq_fts150.stl"/>
                 </geometry>
                 <material name="black"/>
@@ -25,5 +25,5 @@
                 <origin xyz="0 0 0" rpy="0 0 0" />
                 <geometry>
-                    <mesh filename="package://meshes/collision/robotiq_fts150.stl"/>
+                    <mesh filename="package://robotiq_ft_sensor_description/meshes/collision/robotiq_fts150.stl"/>
                 </geometry>
             </collision>

Commit message: feat: change joint name

File: robotiq_ft_sensor_description/urdf/robotiq_ft300.urdf.xacro (robot description, xacro)
@@ -50,5 +50,5 @@
         </link>
          <!-- Connect force sensor with mounting/coupling plate -->
-        <joint name="${tf_prefix}ft300_mounting_plate" type="fixed">
+        <joint name="${tf_prefix}ft300_mounting_plate_joint" type="fixed">
             <origin xyz="0 0 0.0415" rpy="0 ${pi} 0"/>
             <parent link="${tf_prefix}ft300_mounting_plate" />

Commit message: feat: add options from file

File: robotiq_ft_sensor_description/urdf/robotiq_ft300.urdf.xacro (robot description, xacro)
@@ -1,5 +1,5 @@
 <?xml version="1.0"?>
 <robot xmlns:xacro="http://ros.org/wiki/xacro">
-    <xacro:macro name="robotiq_ft300" params="parent tf_prefix *origin">
+    <xacro:macro name="robotiq_ft300" params="parent tf_prefix *origin mesh_from_package:=true">
         <!-- mount the fts to the robot -->
         <joint name="${tf_prefix}ft300_fix" type="fixed">
@@ -18,5 +18,10 @@
                 <origin xyz="0 0 0" rpy="0 0 0" />
                 <geometry>
-                    <mesh filename="package://robotiq_ft_sensor_description/meshes/visual/robotiq_ft300.STL"/>
+                    <xacro:if value="${mesh_from_package}">
+                        <mesh filename="package://robotiq_ft_sensor_description/meshes/visual/robotiq_ft300.STL"/>
+                    </xacro:if>
+                    <xacro:unless value="${mesh_from_package}">
+                        <mesh filename="file://$(find robotiq_ft_sensor_description)/meshes/visual/robotiq_ft300.STL"/>
+                    </xacro:unless>
                 </geometry>
                 <material name="Robotiq-Black">
@@ -27,5 +32,10 @@
                 <origin xyz="0 0 0" rpy="0 0 0" />
                 <geometry>
-                    <mesh filename="package://robotiq_ft_sensor_description/meshes/collision/robotiq_ft300.STL"/>
+                    <xacro:if value="${mesh_from_package}">
+                        <mesh filename="package://robotiq_ft_sensor_description/meshes/collision/robotiq_ft300.STL"/>
+                    </xacro:if>
+                    <xacro:unless value="${mesh_from_package}">
+                        <mesh filename="file://$(find robotiq_ft_sensor_description)/meshes/collision/robotiq_ft300.STL"/>
+                    </xacro:unless>
                 </geometry>
             </collision>
@@ -36,5 +46,10 @@
                 <origin xyz="0 0 0" rpy="0 0 0" />
                 <geometry>
-                    <mesh filename="package://robotiq_ft_sensor_description/meshes/visual/mountings/robotiq_ft300-G-062-COUPLING_G-50-4M6-1D6_20181119.STL"/>
+                    <xacro:if value="${mesh_from_package}">
+                        <mesh filename="package://robotiq_ft_sensor_description/meshes/visual/mountings/robotiq_ft300-G-062-COUPLING_G-50-4M6-1D6_20181119.STL"/>
+                    </xacro:if>
+                    <xacro:unless value="${mesh_from_package}">
+                        <mesh filename="file://$(find robotiq_ft_sensor_description)/meshes/visual/mountings/robotiq_ft300-G-062-COUPLING_G-50-4M6-1D6_20181119.STL"/>
+                    </xacro:unless>
                 </geometry>
                 <material name="Robotiq-Grey">
@@ -45,5 +60,10 @@
                 <origin xyz="0 0 0" rpy="0 0 0" />
                 <geometry>
-                    <mesh filename="package://robotiq_ft_sensor_description/meshes/collision/mountings/robotiq_ft300-G-062-COUPLING_G-50-4M6-1D6_20181119.STL"/>
+                    <xacro:if value="${mesh_from_package}">
+                        <mesh filename="package://robotiq_ft_sensor_description/meshes/collision/mountings/robotiq_ft300-G-062-COUPLING_G-50-4M6-1D6_20181119.STL"/>
+                    </xacro:if>
+                    <xacro:unless value="${mesh_from_package}">
+                        <mesh filename="file://$(find robotiq_ft_sensor_description)/meshes/collision/mountings/robotiq_ft300-G-062-COUPLING_G-50-4M6-1D6_20181119.STL"/>
+                    </xacro:unless>
                 </geometry>
             </collision>

Commit message: feat: reduce inerial

File: robotiq_ft_sensor_description/urdf/robotiq_ft300.urdf.xacro (robot description, xacro)
@@ -11,8 +11,13 @@
         <link name="${tf_prefix}ft300_sensor">
             <inertial>
+                <origin xyz="0 0 0" rpy="0 0 0"/>
+                <mass value="0.001"/>
+                <inertia ixx="0.0001" ixy="0" ixz="0" iyy="0.0001" iyx="0" iyz="0" izz="0.0001" izx="0" izy="0"/>
+            </inertial>
+            <!-- <inertial>
                 <origin xyz="0 0 ${-17 / 1000}" rpy="0 0 0"/>
                 <mass value="0.300"/>
                 <inertia ixx="${262 / 1000000}" ixy="0" ixz="${1 / 1000000}" iyy="${265 / 1000000}" iyx="0" iyz="${1 / 1000000}" izz="${219 / 1000000}" izx="${-1 / 1000000}" izy="${1 / 1000000}"/>
-            </inertial>
+            </inertial> -->
             <visual>
                 <origin xyz="0 0 0" rpy="0 0 0" />

Commit message: feat: robotiq inertia back disable gravity

File: robotiq_ft_sensor_description/urdf/robotiq_ft300.urdf.xacro (robot description, xacro)
@@ -1,45 +1,56 @@
 <?xml version="1.0"?>
 <robot xmlns:xacro="http://ros.org/wiki/xacro">
-    <xacro:macro name="robotiq_ft300" params="parent tf_prefix *origin mesh_from_package:=true">
+    <xacro:macro name="robotiq_ft300"
+                 params="parent tf_prefix *origin mesh_from_package:=true">
         <!-- mount the fts to the robot -->
-        <joint name="${tf_prefix}ft300_fix" type="fixed">
+        <joint name="${tf_prefix}ft300_fix"
+               type="fixed">
             <xacro:insert_block name="origin" />
             <parent link="${tf_prefix}${parent}" />
             <child link="${tf_prefix}ft300_mounting_plate" />
         </joint>
+        <gazebo reference="${tf_prefix}ft300_sensor">
+            <gravity>false</gravity>
+        </gazebo>
         <!-- Link representing the FT300 force-torque sensor -->
         <link name="${tf_prefix}ft300_sensor">
             <inertial>
-                <origin xyz="0 0 0" rpy="0 0 0"/>
-                <mass value="0.001"/>
-                <inertia ixx="0.0001" ixy="0" ixz="0" iyy="0.0001" iyx="0" iyz="0" izz="0.0001" izx="0" izy="0"/>
+                <origin xyz="0 0 ${-17 / 1000}"
+                        rpy="0 0 0" />
+                <mass value="0.300" />
+                <inertia ixx="${262 / 1000000}"
+                         ixy="0"
+                         ixz="${1 / 1000000}"
+                         iyy="${265 / 1000000}"
+                         iyx="0"
+                         iyz="${1 / 1000000}"
+                         izz="${219 / 1000000}"
+                         izx="${-1 / 1000000}"
+                         izy="${1 / 1000000}" />
             </inertial>
-            <!-- <inertial>
-                <origin xyz="0 0 ${-17 / 1000}" rpy="0 0 0"/>
-                <mass value="0.300"/>
-                <inertia ixx="${262 / 1000000}" ixy="0" ixz="${1 / 1000000}" iyy="${265 / 1000000}" iyx="0" iyz="${1 / 1000000}" izz="${219 / 1000000}" izx="${-1 / 1000000}" izy="${1 / 1000000}"/>
-            </inertial> -->
             <visual>
-                <origin xyz="0 0 0" rpy="0 0 0" />
+                <origin xyz="0 0 0"
+                        rpy="0 0 0" />
                 <geometry>
                     <xacro:if value="${mesh_from_package}">
-                        <mesh filename="package://robotiq_ft_sensor_description/meshes/visual/robotiq_ft300.STL"/>
+                        <mesh filename="package://robotiq_ft_sensor_description/meshes/visual/robotiq_ft300.STL" />
                     </xacro:if>
                     <xacro:unless value="${mesh_from_package}">
-                        <mesh filename="file://$(find robotiq_ft_sensor_description)/meshes/visual/robotiq_ft300.STL"/>
+                        <mesh filename="file://$(find robotiq_ft_sensor_description)/meshes/visual/robotiq_ft300.STL" />
                     </xacro:unless>
                 </geometry>
                 <material name="Robotiq-Black">
-                    <color rgba="0.2 0.2 0.2 1.0"/>
+                    <color rgba="0.2 0.2 0.2 1.0" />
                 </material>
             </visual>
             <collision>
-                <origin xyz="0 0 0" rpy="0 0 0" />
+                <origin xyz="0 0 0"
+                        rpy="0 0 0" />
                 <geometry>
                     <xacro:if value="${mesh_from_package}">
-                        <mesh filename="package://robotiq_ft_sensor_description/meshes/collision/robotiq_ft300.STL"/>
+                        <mesh filename="package://robotiq_ft_sensor_description/meshes/collision/robotiq_ft300.STL" />
                     </xacro:if>
                     <xacro:unless value="${mesh_from_package}">
-                        <mesh filename="file://$(find robotiq_ft_sensor_description)/meshes/collision/robotiq_ft300.STL"/>
+                        <mesh filename="file://$(find robotiq_ft_sensor_description)/meshes/collision/robotiq_ft300.STL" />
                     </xacro:unless>
                 </geometry>
@@ -49,41 +60,47 @@
         <link name="${tf_prefix}ft300_mounting_plate">
             <visual>
-                <origin xyz="0 0 0" rpy="0 0 0" />
+                <origin xyz="0 0 0"
+                        rpy="0 0 0" />
                 <geometry>
                     <xacro:if value="${mesh_from_package}">
-                        <mesh filename="package://robotiq_ft_sensor_description/meshes/visual/mountings/robotiq_ft300-G-062-COUPLING_G-50-4M6-1D6_20181119.STL"/>
+                        <mesh filename="package://robotiq_ft_sensor_description/meshes/visual/mountings/robotiq_ft300-G-062-COUPLING_G-50-4M6-1D6_20181119.STL" />
                     </xacro:if>
                     <xacro:unless value="${mesh_from_package}">
-                        <mesh filename="file://$(find robotiq_ft_sensor_description)/meshes/visual/mountings/robotiq_ft300-G-062-COUPLING_G-50-4M6-1D6_20181119.STL"/>
+                        <mesh filename="file://$(find robotiq_ft_sensor_description)/meshes/visual/mountings/robotiq_ft300-G-062-COUPLING_G-50-4M6-1D6_20181119.STL" />
                     </xacro:unless>
                 </geometry>
                 <material name="Robotiq-Grey">
-                    <color rgba="0.4 0.4 0.4 1.0"/>
+                    <color rgba="0.4 0.4 0.4 1.0" />
                 </material>
             </visual>
             <collision>
-                <origin xyz="0 0 0" rpy="0 0 0" />
+                <origin xyz="0 0 0"
+                        rpy="0 0 0" />
                 <geometry>
                     <xacro:if value="${mesh_from_package}">
-                        <mesh filename="package://robotiq_ft_sensor_description/meshes/collision/mountings/robotiq_ft300-G-062-COUPLING_G-50-4M6-1D6_20181119.STL"/>
+                        <mesh filename="package://robotiq_ft_sensor_description/meshes/collision/mountings/robotiq_ft300-G-062-COUPLING_G-50-4M6-1D6_20181119.STL" />
                     </xacro:if>
                     <xacro:unless value="${mesh_from_package}">
-                        <mesh filename="file://$(find robotiq_ft_sensor_description)/meshes/collision/mountings/robotiq_ft300-G-062-COUPLING_G-50-4M6-1D6_20181119.STL"/>
+                        <mesh filename="file://$(find robotiq_ft_sensor_description)/meshes/collision/mountings/robotiq_ft300-G-062-COUPLING_G-50-4M6-1D6_20181119.STL" />
                     </xacro:unless>
                 </geometry>
             </collision>
         </link>
-         <!-- Connect force sensor with mounting/coupling plate -->
-        <joint name="${tf_prefix}ft300_mounting_plate_joint" type="fixed">
-            <origin xyz="0 0 0.0415" rpy="0 ${pi} 0"/>
+        <!-- Connect force sensor with mounting/coupling plate -->
+        <joint name="${tf_prefix}ft300_mounting_plate_joint"
+               type="fixed">
+            <origin xyz="0 0 0.0415"
+                    rpy="0 ${pi} 0" />
             <parent link="${tf_prefix}ft300_mounting_plate" />
             <child link="${tf_prefix}ft300_sensor" />
         </joint>
-        <joint name="${tf_prefix}measurment_joint" type="fixed">
-            <origin xyz="0 0 0" rpy="0 ${pi} ${-pi/2}" />
+        <joint name="${tf_prefix}measurment_joint"
+               type="fixed">
+            <origin xyz="0 0 0"
+                    rpy="0 ${pi} ${-pi/2}" />
             <parent link="${tf_prefix}ft300_sensor" />
             <child link="${tf_prefix}robotiq_ft_frame_id" />
         </joint>
-        <link name="${tf_prefix}robotiq_ft_frame_id"/>
+        <link name="${tf_prefix}robotiq_ft_frame_id" />
     </xacro:macro>
 </robot>
